File: hardware/happytuesdays.brd (EAGLE design)
At the start: 40 x 40 mm, 29 parts, among them IC1 4028D, IC2 4028D

Commit message: Board finished, added partslist
Parts:
- removed U$8: CRYSTAL2.5X2, NordicSemi:2.5X2MM
- added C11, C12: 12pF, microbuilder_v3:_0402
- added C14, C19, C20: 1µF, resistor:C0603K
- added CN1: (no value), microbuilder:JSTPH2
- added IC4: TLV70033DCK, tlv700:SC70-5L
- added IC5: MAX1555, SparkFun:SOT23-5
- added LED1, LED2: (no value), led:CHIPLED_0603
- added R1, R2: 1kΩ, microbuilder_v3:_0402
- added X1: USB-MICROB, SparkFun:USB-MICROB
- added Y1: CRYSTAL2.5X2, NordicSemi:2.5X2MM
- RN1, RN2, RN3, RN4: value (none) -> 68Ω
- moved JTAG1 20.3 mm to (35.8, 4.25)
- moved C2 5.71 mm to (20.2, 26.0), turned to 135 degrees
- moved C1 2.43 mm to (27.8, 18.9)
- moved C6 2.26 mm to (27.0, 25.8)
- moved L2 1.88 mm to (26.4, 19.9), turned to 270 degrees
- moved C4 1.67 mm to (26.1, 23.9)
- moved C9 1.63 mm to (15.6, 23.8), turned to 180 degrees
- moved L3 1.46 mm to (25.5, 25.2), turned to 90 degrees
- moved C10 1.41 mm to (14.2, 18.0), turned to 90 degrees
- moved C8 1.38 mm to (12.8, 23.8), turned to 180 degrees
- moved L4 1.23 mm to (13.8, 22.8)
- moved L5 1.23 mm to (15.5, 22.2), turned to 270 degrees
- moved L1 1.00 mm to (25.5, 20.4)
- moved C15 0.80 mm to (24.5, 23.4), turned to 90 degrees
- moved C7 0.75 mm to (27.0, 26.8)
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- renumbered U$1 to IC3
Connections:
- net N$2 renamed DCC
- removed net N$3: IC3.38
- removed net N$4: IC3.37
- new net 5.0V: C20.1, IC5.4, X1.VBUS
- new net BATT: C19.1, CN1.2, IC4.1, IC4.3, IC5.5, LED1.A
- new net CHG: IC5.3, R2.1
- new net LED: LED1.C, R2.2
- new net N$6: IC3.14, R1.2
- new net N$8: LED2.A, R1.1
- new net X1: C12.1, IC3.37, Y1.X1
- new net X2: C11.2, IC3.38, Y1.X2
- net 3.3V: now also C14.1, IC4.5
- net GND: now also C11.1, C12.2, C14.2, C19.2, C20.2, CN1.1, IC4.2, IC5.2, LED2.C, X1.GND, Y1.GND, Y1.GND2
Routing:
- net 3.3V: track 0.00 -> 110.8 mm, vias 0 -> 6
- net ANT: track 0.00 -> 31.1 mm
- net BATT: track 0.00 -> 28.9 mm, vias 0 -> 3
- net SWDCLK: track 0.00 -> 27.1 mm
- net SWDIO: track 1.79 -> 25.9 mm
- net AVDD: track 0.00 -> 16.2 mm, vias 0 -> 2
- net 2Q8: track 0.00 -> 10.6 mm, vias 0 -> 2
- net 1Q8: track 0.00 -> 10.6 mm, vias 0 -> 2
- net X1: track 0.00 -> 6.58 mm
- net GND: track 0.00 -> 5.12 mm, vias 9 -> 43
- net 5.0V: track 0.00 -> 4.95 mm
- net VDD_PA: track 0.00 -> 4.68 mm
- net X2: track 0.00 -> 4.66 mm
- net DEC2: track 0.00 -> 4.48 mm
- net ANT2: track 0.00 -> 3.54 mm
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
Commit message: Added partlist
Parts:
- removed C19, C20: 1µF, resistor:C0603K
- added C13: 100nF, microbuilder_v3:_0402
- added C16: 1µF, resistor:C0603K
- C15: value 100nF -> 1µF; device microbuilder_v3:_0402 -> resistor:C0603K
- L3: value 3.3nF -> 3.3nH
- moved C14 17.2 mm to (27.0, 7.50), turned to 0 degrees
- moved C15 15.3 mm to (15.5, 11.0), turned to 0 degrees
Connections:
- net 3.3V: now also C16.1; no longer C14.1
- net 5.0V: now also C14.1; no longer C20.1
- net AVDD: now also C13.1; no longer C15.1
- net BATT: now also C15.1; no longer C19.1
- net GND: now also C13.2, C16.2; no longer C19.2, C20.2
Changed lines of the file:
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@@
 <element name="IC3" library="NordicSemi" package="QFN48" value="NRF51822" x="20" y="20"/>
 <element name="JTAG1" library="microbuilder_v3" package="2X05_1.27MM_SMT" value="" x="35.75" y="4.25" rot="R270"/>
-<element name="C15" library="microbuilder_v3" package="_0402" value="100nF" x="24.5" y="23.375" rot="R90"/>
+<element name="C13" library="microbuilder_v3" package="_0402" value="100nF" x="24.5" y="23.375" rot="R90"/>
 <element name="C1" library="microbuilder_v3" package="_0402" value="47nF" x="27.75" y="18.875"/>
 <element name="C2" library="microbuilder_v3" package="_0402" value="100nF" x="20.25" y="26" rot="R135"/>
@@
 <element name="C6" library="microbuilder_v3" package="_0402" value="1.5pF" x="27" y="25.75"/>
 <element name="C7" library="microbuilder_v3" package="_0402" value="1.5pF" x="27" y="26.75"/>
-<element name="L3" library="microbuilder_v3" package="_0402" value="3.3nF" x="25.5" y="25.25" rot="R90"/>
+<element name="L3" library="microbuilder_v3" package="_0402" value="3.3nH" x="25.5" y="25.25" rot="R90"/>
 <element name="L4" library="microbuilder_v3" package="_0402" value="10µH" x="13.75" y="22.75"/>
 <element name="L5" library="microbuilder_v3" package="_0402" value="15nH" x="15.5" y="22.25" rot="R270"/>
@@
 <element name="C12" library="microbuilder_v3" package="_0402" value="12pF" x="23.25" y="29.25" rot="R135"/>
 <element name="IC4" library="tlv700" package="SC70-5L" value="TLV70033DCK" x="14" y="14"/>
-<element name="C14" library="resistor" package="C0603K" value="1µF" x="13" y="17.5" rot="R90"/>
+<element name="C16" library="resistor" package="C0603K" value="1µF" x="13" y="17.5" rot="R90"/>
 <element name="IC5" library="SparkFun" package="SOT23-5" value="MAX1555" x="22" y="7" rot="R270"/>
 <element name="CN1" library="microbuilder" package="JSTPH2" value="" x="15.5" y="4" rot="R180"/>
-<element name="C19" library="resistor" package="C0603K" value="1µF" x="15.5" y="11"/>
-<element name="C20" library="resistor" package="C0603K" value="1µF" x="27" y="7.5"/>
+<element name="C15" library="resistor" package="C0603K" value="1µF" x="15.5" y="11"/>
+<element name="C14" library="resistor" package="C0603K" value="1µF" x="27" y="7.5"/>
 <element name="LED1" library="led" package="CHIPLED_0603" value="" x="21.25" y="2"/>
 <element name="X1" library="SparkFun" package="USB-MICROB" value="USB-MICROB" x="27" y="2.5"/>
@@
 <contactref element="IC3" pad="34"/>
 <contactref element="IC3" pad="33"/>
-<contactref element="C15" pad="2"/>
+<contactref element="C13" pad="2"/>
 <contactref element="C1" pad="2"/>
 <contactref element="C2" pad="2"/>
@@
 <via x="34.25" y="15.125" extent="1-16" drill="0.3"/>
 <contactref element="IC4" pad="2"/>
+<contactref element="C16" pad="2"/>
+<contactref element="IC5" pad="2"/>
+<contactref element="C15" pad="2"/>
 <contactref element="C14" pad="2"/>
-<contactref element="IC5" pad="2"/>
-<contactref element="C19" pad="2"/>
-<contactref element="C20" pad="2"/>
 <contactref element="CN1" pad="1"/>
 <contactref element="X1" pad="GND"/>
@@
 <contactref element="IC3" pad="35"/>
 <contactref element="IC3" pad="36"/>
-<contactref element="C15" pad="1"/>
+<contactref element="C13" pad="1"/>
 <contactref element="L4" pad="1"/>
 <contactref element="C8" pad="1"/>
@@
 <contactref element="IC1" pad="16"/>
 <contactref element="IC4" pad="5"/>
-<contactref element="C14" pad="1"/>
+<contactref element="C16" pad="1"/>
 <wire x1="13.35" y1="14.85" x2="13.35" y2="16.275" width="0.4" layer="1"/>
 <wire x1="13.35" y1="16.275" x2="13" y2="16.625" width="0.4" layer="1"/>
@@
 <signal name="5.0V">
 <contactref element="IC5" pad="4"/>
-<contactref element="C20" pad="1"/>
+<contactref element="C14" pad="1"/>
 <contactref element="X1" pad="VBUS"/>
 <wire x1="26.125" y1="7.5" x2="25.7" y2="7.075" width="0.4" layer="1"/>
@@
 </signal>
 <signal name="BATT">
-<contactref element="C19" pad="1"/>
+<contactref element="C15" pad="1"/>
 <contactref element="IC5" pad="5"/>
 <contactref element="CN1" pad="2"/>
