File: hardware/happytuesdays.sch (EAGLE design)
At the start: 29 parts, among them IC1 4028D, IC2 4028D

Commit message: Board finished, added partslist
Parts:
- removed U$1: NRF51822, NordicSemi:NRF51822
- removed U$8: CRYSTAL2.5X2, NordicSemi:CRYSTAL2.5X2
- added C11, C12: 12pF, microbuilder_v3:CAP_CERAMIC_0402
- added C14, C19, C20: 1µF, resistor:C-EUC0603K
- added CN1: (no value), microbuilder:JST_2PIN
- added IC3: NRF51822, NordicSemi:NRF51822
- added IC4: TLV70033DCK, tlv700:TLV700DCK
- added IC5: MAX1555, SparkFun:MAX1555
- added LED1, LED2: (no value), led:LEDCHIPLED_0603
- added R1, R2: 1kΩ, microbuilder_v3:RESISTOR_0402
- added X1: USB-MICROB, SparkFun:USB-MICROB
- added Y1: CRYSTAL2.5X2, NordicSemi:CRYSTAL2.5X2
- RN1, RN2, RN3, RN4: value (none) -> 68Ω
Connections:
- removed net N$2: L5.2, U$1.DCC
- removed net N$3: U$1.XC2
- removed net N$4: U$1.XC1
- new net 5.0V: C20.1, IC5.DC, X1.VBUS
- new net BATT: C19.1, CN1.2, IC4.EN, IC4.IN, IC5.BATT, LED1.A
- new net CHG: IC5.CHG, R2.1
- new net DCC: IC3.DCC, L5.2
- new net LED: LED1.C, R2.2
- new net N$6: IC3.P0.08, R1.2
- new net N$8: LED2.A, R1.1
- new net X1: C12.P$1, IC3.XC1, Y1.X1
- new net X2: C11.P$2, IC3.XC2, Y1.X2
- net 1A: now also IC3.P0.17; no longer U$1.P0.17
- net 1B: now also IC3.P0.20; no longer U$1.P0.20
- net 1C: now also IC3.P0.19; no longer U$1.P0.19
- net 1C1: now also IC3.P0.16; no longer U$1.P0.16
- net 1C2: now also IC3.P0.15; no longer U$1.P0.15
- net 1C3: now also IC3.P0.14; no longer U$1.P0.14
- net 1C4: now also IC3.P0.13; no longer U$1.P0.13
- net 1C5: now also IC3.P0.12; no longer U$1.P0.12
- net 1C6: now also IC3.P0.11; no longer U$1.P0.11
- net 1C7: now also IC3.P0.10; no longer U$1.P0.10
- net 1C8: now also IC3.P0.09; no longer U$1.P0.09
- net 1D: now also IC3.P0.18; no longer U$1.P0.18
- net 2A: now also IC3.P0.00; no longer U$1.P0.00
- net 2B: now also IC3.P0.03; no longer U$1.P0.03
- net 2C: now also IC3.P0.02; no longer U$1.P0.02
- net 2C1: now also IC3.P0.29; no longer U$1.P0.29
- net 2C2: now also IC3.P0.28; no longer U$1.P0.28
- net 2C3: now also IC3.P0.27; no longer U$1.P0.27
- net 2C4: now also IC3.P0.26; no longer U$1.P0.26
- net 2C5: now also IC3.P0.25; no longer U$1.P0.25
- net 2C6: now also IC3.P0.24; no longer U$1.P0.24
- net 2C7: now also IC3.P0.23; no longer U$1.P0.23
- net 2C8: now also IC3.P0.22; no longer U$1.P0.22
- net 2D: now also IC3.P0.01; no longer U$1.P0.01
- net 3.3V: now also C14.1, IC3.VDD, IC3.VDD_2, IC4.OUT; no longer U$1.VDD, U$1.VDD_2
- net ANT1: now also IC3.ANT1; no longer U$1.ANT1
- net ANT2: now also IC3.ANT2; no longer U$1.ANT2
- net AVDD: now also IC3.AVDD, IC3.AVDD_2; no longer U$1.AVDD, U$1.AVDD_2
- net DEC1: now also IC3.DEC1; no longer U$1.DEC1
- net DEC2: now also IC3.DEC2; no longer U$1.DEC2
- net GND: now also C11.P$1, C12.P$2, C14.2, C19.2, C20.2, CN1.1, IC3.DIE_PAD, IC3.VSS, IC3.VSS_2, IC3.VSS_3, IC4.GND, IC5.GND, LED2.C, X1.GND, Y1.GND, Y1.GND2; no longer U$1.DIE_PAD, U$1.VSS, U$1.VSS_2, U$1.VSS_3
- net SWDCLK: now also IC3.SWDCLK; no longer U$1.SWDCLK
- net SWDIO: now also IC3.SWDIO/NRESET; no longer U$1.SWDIO/NRESET
- net VDD_PA: now also IC3.VDD_PA; no longer U$1.VDD_PA
Other:
- note added: "TLV70033"
- moved on the sheet: C1, C10, C15, C2, C3, C4, C5, C6, C7, C8, C9, IC1P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

Commit message: Added partlist
Parts:
- removed C19, C20: 1µF, resistor:C-EUC0603K
- added C13: 100nF, microbuilder_v3:CAP_CERAMIC_0402
- added C16: 1µF, resistor:C-EUC0603K
- C15: value 100nF -> 1µF; device microbuilder_v3:CAP_CERAMIC_0402 -> resistor:C-EUC0603K
- L3: value 3.3nF -> 3.3nH
Connections:
- net 3.3V: now also C16.1; no longer C14.1
- net 5.0V: now also C14.1; no longer C20.1
- net AVDD: now also C13.P$1; no longer C15.P$1
- net BATT: now also C15.1; no longer C19.1
- net GND: now also C13.P$2, C15.2, C16.2; no longer C15.P$2, C19.2, C20.2
Other:
- moved on the sheet: C14, C15
Changed lines of the file:
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@@
 <part name="U$2" library="microbuilder_v3" deviceset="AVDD" device=""/>
 <part name="U$3" library="microbuilder_v3" deviceset="AVDD" device=""/>
-<part name="C15" library="microbuilder_v3" deviceset="CAP_CERAMIC" device="_0402" value="100nF"/>
+<part name="C13" library="microbuilder_v3" deviceset="CAP_CERAMIC" device="_0402" value="100nF"/>
 <part name="C1" library="microbuilder_v3" deviceset="CAP_CERAMIC" device="_0402" value="47nF"/>
 <part name="GND3" library="SparkFun" deviceset="GND" device=""/>
@@
 <part name="C6" library="microbuilder_v3" deviceset="CAP_CERAMIC" device="_0402" value="1.5pF"/>
 <part name="C7" library="microbuilder_v3" deviceset="CAP_CERAMIC" device="_0402" value="1.5pF"/>
-<part name="L3" library="microbuilder_v3" deviceset="INDUCTOR" device="_0402" value="3.3nF"/>
+<part name="L3" library="microbuilder_v3" deviceset="INDUCTOR" device="_0402" value="3.3nH"/>
 <part name="GND7" library="SparkFun" deviceset="GND" device=""/>
 <part name="GND8" library="SparkFun" deviceset="GND" device=""/>
@@
 <part name="IC4" library="tlv700" deviceset="TLV700" device="DCK" value="TLV70033DCK"/>
 <part name="U$22" library="microbuilder" deviceset="GND" device=""/>
-<part name="C14" library="resistor" deviceset="C-EU" device="C0603K" value="1µF"/>
+<part name="C16" library="resistor" deviceset="C-EU" device="C0603K" value="1µF"/>
 <part name="U$25" library="microbuilder" deviceset="GND" device=""/>
 <part name="U$31" library="microbuilder_v3" deviceset="3.3V" device=""/>
 <part name="IC5" library="SparkFun" deviceset="MAX1555" device=""/>
 <part name="CN1" library="microbuilder" deviceset="JST_2PIN" device=""/>
-<part name="C19" library="resistor" deviceset="C-EU" device="C0603K" value="1µF"/>
-<part name="C20" library="resistor" deviceset="C-EU" device="C0603K" value="1µF"/>
+<part name="C15" library="resistor" deviceset="C-EU" device="C0603K" value="1µF"/>
+<part name="C14" library="resistor" deviceset="C-EU" device="C0603K" value="1µF"/>
 <part name="U$32" library="microbuilder" deviceset="GND" device=""/>
 <part name="U$33" library="microbuilder" deviceset="GND" device=""/>
@@
 <instance part="U$2" gate="G$1" x="129.54" y="139.7"/>
 <instance part="U$3" gate="G$1" x="10.16" y="142.24"/>
-<instance part="C15" gate="G$1" x="124.46" y="129.54"/>
+<instance part="C13" gate="G$1" x="124.46" y="129.54"/>
 <instance part="C1" gate="G$1" x="129.54" y="104.14"/>
 <instance part="GND3" gate="1" x="129.54" y="99.06"/>
@@
 <instance part="IC4" gate="G$1" x="215.9" y="58.42"/>
 <instance part="U$22" gate="G$1" x="223.52" y="43.18"/>
-<instance part="C14" gate="G$1" x="241.3" y="53.34"/>
+<instance part="C16" gate="G$1" x="241.3" y="53.34"/>
 <instance part="U$25" gate="G$1" x="241.3" y="43.18"/>
 <instance part="U$31" gate="G$1" x="241.3" y="71.12"/>
 <instance part="IC5" gate="G$1" x="170.18" y="60.96"/>
 <instance part="CN1" gate="G$1" x="205.74" y="71.12" rot="R90"/>
-<instance part="C19" gate="G$1" x="198.12" y="53.34"/>
-<instance part="C20" gate="G$1" x="190.5" y="53.34"/>
+<instance part="C15" gate="G$1" x="198.12" y="53.34"/>
+<instance part="C14" gate="G$1" x="190.5" y="53.34"/>
 <instance part="U$32" gate="G$1" x="190.5" y="43.18"/>
 <instance part="U$33" gate="G$1" x="198.12" y="43.18"/>
@@
 <wire x1="121.92" y1="127" x2="124.46" y2="127" width="0.1524" layer="91"/>
 <junction x="121.92" y="127"/>
-<pinref part="C15" gate="G$1" pin="P$2"/>
+<pinref part="C13" gate="G$1" pin="P$2"/>
 <junction x="124.46" y="127"/>
 <wire x1="124.46" y1="127" x2="129.54" y2="127" width="0.1524" layer="91"/>
@@
 <segment>
 <pinref part="U$25" gate="G$1" pin="GND"/>
-<pinref part="C14" gate="G$1" pin="2"/>
+<pinref part="C16" gate="G$1" pin="2"/>
 <wire x1="241.3" y1="45.72" x2="241.3" y2="48.26" width="0.1524" layer="91"/>
 </segment>
@@
 <segment>
 <wire x1="198.12" y1="48.26" x2="198.12" y2="45.72" width="0.1524" layer="91"/>
-<pinref part="C19" gate="G$1" pin="2"/>
+<pinref part="C15" gate="G$1" pin="2"/>
 <pinref part="U$33" gate="G$1" pin="GND"/>
 </segment>
 <segment>
 <wire x1="190.5" y1="48.26" x2="190.5" y2="45.72" width="0.1524" layer="91"/>
-<pinref part="C20" gate="G$1" pin="2"/>
+<pinref part="C14" gate="G$1" pin="2"/>
 <pinref part="U$32" gate="G$1" pin="GND"/>
 </segment>
@@
 <wire x1="129.54" y1="134.62" x2="129.54" y2="137.16" width="0.1524" layer="91"/>
 <junction x="121.92" y="134.62"/>
-<pinref part="C15" gate="G$1" pin="P$1"/>
+<pinref part="C13" gate="G$1" pin="P$1"/>
 <junction x="124.46" y="134.62"/>
 </segment>
@@
 <segment>
 <pinref part="IC4" gate="G$1" pin="OUT"/>
-<pinref part="C14" gate="G$1" pin="1"/>
+<pinref part="C16" gate="G$1" pin="1"/>
 <wire x1="236.22" y1="63.5" x2="241.3" y2="63.5" width="0.1524" layer="91"/>
 <wire x1="241.3" y1="63.5" x2="241.3" y2="55.88" width="0.1524" layer="91"/>
@@
 <junction x="190.5" y="58.42"/>
 <pinref part="IC5" gate="G$1" pin="DC"/>
-<pinref part="C20" gate="G$1" pin="1"/>
+<pinref part="C14" gate="G$1" pin="1"/>
 <pinref part="U$36" gate="G$1" pin="5.0V"/>
 </segment>
@@
 <junction x="205.74" y="63.5"/>
 <label x="182.88" y="63.5" size="1.778" layer="95"/>
-<pinref part="C19" gate="G$1" pin="1"/>
+<pinref part="C15" gate="G$1" pin="1"/>
 <pinref part="IC5" gate="G$1" pin="BATT"/>
 <pinref part="CN1" gate="G$1" pin="2"/>
